Commit message: New4-wheeled Robot made. currently not moving

File: urdf/robot.urdf (robot description, URDF)
Before this commit: robot udacity_bot, 5 links, 4 joints
Links:
- removed link left_wheel
- removed link right_wheel
- added link hokuyo, mass 0.1; collision box size=.05 .05 .05; visual mesh filename=package://udacity_bot/meshes/hokuyo.dae
- added link leftb_wheel, mass 0.033; collision cylinder length=0.025 radius=0.0335; visual cylinder length=0.025 radius=0.0335
- added link leftf_wheel, mass 0.033; collision cylinder length=0.025 radius=0.03; visual cylinder length=0.025 radius=0.0335
- added link rightb_wheel, mass 0.033; collision cylinder length=0.025 radius=0.0335; visual cylinder length=0.025 radius=0.0335
- added link rightf_wheel, mass 0.033; collision cylinder length=0.025 radius=0.0335; visual cylinder length=0.025 radius=0.0335
- link camera: geometry collision box size=.005 .005 .005; visual box size=.05 .05 .05
- link chassis: mass 15.0 -> 0.489; geometry collision box size=.24 .1 .02; visual box size=.24 .1 .02
Joints:
- removed joint left_wheel_hinge
- removed joint right_wheel_hinge
- added joint hokuyo_joint: type fixed, parent chassis, child hokuyo, origin xyz=-0.005 0 0.127 rpy=0 0 0
- added joint left__back_wheel_hinge: type continuous, parent chassis, child leftb_wheel, origin xyz=0.06 -0.07 0 rpy=1.570796 0 0, axis 0 1 0, limit effort=10000 velocity=1000
- added joint left__front_wheel_hinge: type continuous, parent chassis, child leftf_wheel, origin xyz=-0.06 -0.07 0 rpy=1.570796 0 0, axis 0 1 0, limit effort=10000 velocity=1000
- added joint right_back_wheel_hinge: type continuous, parent chassis, child rightb_wheel, origin xyz=0.06 0.07 0 rpy=1.570796 0 0, axis 0 1 0, limit effort=10000 velocity=1000
- added joint right_front_wheel_hinge: type continuous, parent chassis, child rightf_wheel, origin xyz=-0.06 0.07 0 rpy=1.570796 0 0, axis 0 1 0, limit effort=10000 velocity=1000
- joint camera_joint: axis (none) -> 0 0 0; origin xyz=0.2 0.0 0 rpy=0 0 0 -> xyz=0 0 0.119 rpy=0 0 0; type rigid -> fixed

File: urdf/udacity_bot.xacro (robot description, xacro)
@@ -9,136 +9,137 @@
   </joint>
   <link name='chassis'>
-    <pose>0 0 0.1 0 0 0</pose>
-    <inertial>
-      <mass value="15.0"/>
-      <origin xyz="0.0 0 0" rpy=" 0 0 0"/>
-      <inertia
-          ixx="0.1" ixy="0" ixz="0"
-          iyy="0.1" iyz="0"
-          izz="0.1"
-      />
-    </inertial>
-    <collision name='collision'>
-      <origin xyz="0 0 0" rpy=" 0 0 0"/>
-      <geometry>
-        <box size=".4 .2 .1"/>
-      </geometry>
-    </collision>
-    <visual name='chassis_visual'>
-      <origin xyz="0 0 0" rpy=" 0 0 0"/>
-      <geometry>
-        <box size=".4 .2 .1"/>
-      </geometry>
-    </visual>
-    <visual name='back_caster_visual'>
-      <origin xyz="-0.15 0 -0.05" rpy=" 0 0 0"/>
-      <geometry>
-        <sphere radius="0.05"/>
-      </geometry>
-    </visual>
-    <collision name='back_caster_collision'>
-	<origin xyz="-0.15 0 -0.05" rpy=" 0 0 0"/>
-      	<geometry>
-          <sphere radius="0.0499"/>
-      	</geometry>
-      <surface>
-        <friction>
-          <ode>
-            <mu>0</mu>
-            <mu2>0</mu2>
-            <slip1>1.0</slip1>
-            <slip2>1.0</slip2>
-          </ode>
-        </friction>
+	<pose>0 0 0.1 0 0 0</pose>
+	<inertial>
+		<mass value="0.5"/>
+		<origin xyz="0.0 0 0" rpy=" 0 0 0"/>
+		<inertia
+			  ixx="0.1" ixy="0" ixz="0"
+			  iyy="0.1" iyz="0"
+			  izz="0.1"
+		/>
+	</inertial>
+	<collision name='chassis_collision'>
+		<origin xyz="0 0 0" rpy=" 0 0 0"/>
+     		<geometry>
+     			<box size=".24 .1 .02"/>
+    		</geometry>
+	</collision>
+	<visual name='chassis_visual'>
+		  <origin xyz="0 0 0" rpy=" 0 0 0"/>
+		  <geometry>
+			<box size=".24 .1 .02"/>
+		  </geometry>
+	</visual>
+		<visual name="rightb_wheel_visual" >
+		<origin xyz="-0.06 0.07 0" rpy="1.570796 0 0"/>
+			  <geometry>
+				<cylinder length="0.025" radius="0.0335"/>
+			  </geometry>
+		</visual>
+		<inertial>
+			  <mass value="0.033"/>
+			  <origin xyz="0.0 0 0" rpy=" 0 0 0"/>
+			  <inertia
+				  ixx="0.1" ixy="0" ixz="0"
+				  iyy="0.1" iyz="0"
+				  izz="0.1"
+			  />
+    	  	</inertial>
+		<collision name="rightb_wheel_collision">
+			<origin xyz="-0.06 0.07 0" rpy="1.570796 0 0"/>
+			  <geometry>
+				<cylinder length="0.025" radius="0.0335"/>
+			  </geometry>
+		 <surface>
+        		<friction>
+         		 <ode>
+         		   <mu>0</mu>
+          		  <mu2>0</mu2>
+           		 <slip1>1.0</slip1>
+          		  <slip2>1.0</slip2>
+         			 </ode>
+       			 </friction>
       </surface>
-    </collision>
-    <collision name='front_caster_collision'>
-      <origin xyz="0.15 0 -0.05" rpy=" 0 0 0"/>
-      <geometry>
-        <sphere radius="0.0499"/>
-      </geometry>
-      <surface>
-        <friction>
-          <ode>
-            <mu>0</mu>
-            <mu2>0</mu2>
-            <slip1>1.0</slip1>
-            <slip2>1.0</slip2>
-          </ode>
-        </friction>
-      </surface>
-    </collision>
-    <visual name='front_caster_visual'>
-      <origin xyz="0.15 0 -0.05" rpy=" 0 0 0"/>
-      <geometry>
-        <sphere radius="0.05"/>
-      </geometry>
-    </visual>
+		</collision>
+		<visual name="leftb_wheel_visual">
+		<origin xyz="-0.06 -0.07 0" rpy="1.570796 0 0"/>
+			  <geometry>
+				<cylinder length="0.025" radius="0.0335"/>
+			  </geometry>
+		</visual>
+		<inertial>
+			  <mass value="0.033"/>
+			  <origin xyz="0.0 0 0" rpy=" 0 0 0"/>
+			  <inertia
+				  ixx="0.1" ixy="0" ixz="0"
+				  iyy="0.1" iyz="0"
+				  izz="0.1"
+			  />
+    		</inertial>
+		<collision name="leftb_wheel_collision">
+		<origin xyz="-0.06 -0.07 0" rpy="1.570796 0 0"/>
+			  <geometry>
+				<cylinder length="0.025" radius="0.0335"/>
+			  </geometry>
+ 			<surface>
+        		 <friction>
+         		 	<ode>
+         		 	  <mu>0</mu>
+          		 	 <mu2>0</mu2>
+           			 <slip1>1.0</slip1>
+          			  <slip2>1.0</slip2>
+         			 </ode>
+       			 </friction>
+      			</surface>
+		</collision>
   </link>
-  <link name="right_wheel">
-    <visual>
-      <origin xyz="0 0 0" rpy="0 1.5707 1.5707"/>
-       <geometry>
-        <cylinder length="0.05" radius="0.1"/>
-      </geometry>
-    </visual>
-    <inertial>
-      <mass value="5.0"/>
-      <origin xyz="0.0 0 0" rpy=" 0 0 0"/>
-      <inertia
-          ixx="0.1" ixy="0" ixz="0"
-          iyy="0.1" iyz="0"
-          izz="0.1"
-      />
-    </inertial>
-	<collision>
-      <origin xyz="0 0 0" rpy="0 1.5707 1.5707"/>
-       <geometry>
-        <cylinder length="0.05" radius="0.1"/>
-      </geometry>
-    </collision>
- </link>
-  <link name="left_wheel">
-    <visual>
-      <origin xyz="0 0 0" rpy="0 1.5707 1.5707"/>
-       <geometry>
-        <cylinder length="0.05" radius="0.1"/>
-      </geometry>
-    </visual>
-    <inertial>
-      <mass value="5.0"/>
-      <origin xyz="0.0 0 0" rpy=" 0 0 0"/>
-      <inertia
-          ixx="0.1" ixy="0" ixz="0"
-          iyy="0.1" iyz="0"
-          izz="0.1"
-      />
-    </inertial>
-	<collision>
-      <origin xyz="0 0 0" rpy="0 1.5707 1.5707"/>
-       <geometry>
-        <cylinder length="0.05" radius="0.1"/>
-      </geometry>
-    </collision>
-  </link>
-<joint type="continuous" name="left_wheel_hinge">
-    <origin xyz="0 0.15 0" rpy="0 0 0"/>
-    <child link="left_wheel"/>
-    <parent link="chassis"/>
-    <axis xyz="0 1 0" rpy="0 0 0"/>
-    <limit effort="10000" velocity="1000"/>
-    <joint_properties damping="1.0" friction="1.0"/>
-  </joint>
-<joint type="continuous" name="right_wheel_hinge">
-    <origin xyz="0 -0.15 0" rpy="0 0 0"/>
-    <child link="right_wheel"/>
-    <parent link="chassis"/>
-    <axis xyz="0 1 0" rpy="0 0 0"/>
-    <limit effort="10000" velocity="1000"/>
-    <joint_properties damping="1.0" friction="1.0"/>
-  </joint>
-<link name="camera">
+	<link name='rightf_wheel'>
+		<visual>
+		 <origin xyz="0.0 0 0" rpy=" 0 0 0"/>
+			  <geometry>
+				<cylinder length="0.025" radius="0.0335"/>
+			  </geometry>
+		</visual>
+		<inertial>
+			  <mass value="0.033"/>
+			  <origin xyz="0.0 0 0" rpy=" 0 0 0"/>
+			  <inertia
+				  ixx="0.1" ixy="0" ixz="0"
+				  iyy="0.1" iyz="0"
+				  izz="0.1"
+			  />
+    		</inertial>
+		<collision>
+		<origin xyz="0.0 0 0" rpy=" 0 0 0"/>
+			  <geometry>
+				<cylinder length="0.025" radius="0.0335"/>
+			  </geometry>
+			</collision>
+	</link>
+	<link name='leftf_wheel'>
+		<visual>
+			  <geometry>
+				<cylinder length="0.025" radius="0.0335"/>
+			  </geometry>
+		</visual>
+		<inertial>
+			  <mass value="0.033"/>
+			  <origin xyz="0.0 0 0" rpy=" 0 0 0"/>
+			  <inertia
+				  ixx="0.1" ixy="0" ixz="0"
+				  iyy="0.1" iyz="0"
+				  izz="0.1"
+			  />
+    		</inertial>
+		<collision>
+			  <origin xyz="0 0 0" rpy=" 0 0 0"/>
+			  <geometry>
+				<cylinder length="0.025" radius="0.03"/>
+			  </geometry>
+		</collision>
+	</link>
+	<link name="camera">
      <visual>
-      <origin xyz="0 0 0" rpy="0 0 0"/>
+     	<origin xyz="0 0 0" rpy="0 0 0"/>
        <geometry>
         <box size=".05 .05 .05"/>
@@ -146,5 +147,5 @@
     </visual>
     <inertial>
-      <mass value="0.1"/>
+      <mass value="0.01"/>
       <origin xyz="0 0 0" rpy=" 0 0 0"/>
       <inertia
@@ -161,9 +162,4 @@
     </collision>
 </link>
-  <joint name="camera_robot_joint" type="fixed">
-    <origin xyz="0.2 0 0" rpy="0 0 0" />
-    <parent link="chassis"/>
-    <child link="camera"/>
-  </joint>
 <link name="hokuyo">
      <visual>
@@ -182,15 +178,37 @@
       />
     </inertial>
-    <collision>
-      <origin xyz="0 0 0" rpy="0 0 0"/>
-       <geometry>
-        <box size=".05 .05 .05"/>
-      </geometry>
-    </collision>
-</link>
-  <joint name="hokuyo_joint" type="fixed">
-    <origin xyz=".15 0 .1 " rpy="0 0 0" />
-    <parent link="chassis"/>
-    <child link="hokuyo"/>
-  </joint>
+	    <collision>
+	      <origin xyz="0 0 0" rpy="0 0 0"/>
+	       <geometry>
+	        <box size=".05 .05 .05"/>
+	      </geometry>
+	    </collision>
+	</link>
+	  <joint name="hokuyo_joint" type="fixed">
+	    <origin xyz="0.13 0 0.127" rpy="0 0 0"/>
+	    <parent link="chassis"/>
+	    <child link="hokuyo"/>
+	  </joint>
+	<joint type="fixed" name="camera_joint">
+		<origin xyz="0.13 0.05 0.07" rpy="0 0 0"/>
+		<child link="camera"/>
+		<parent link="chassis"/>
+		<axis xyz="0 0 0" rpy="0 0 0"/>
+  	</joint>
+	<joint type="continuous" name="left__front_wheel_hinge">
+		<origin xyz="0.06 0.07 0" rpy="1.570796 0 0"/>
+		<child link="leftf_wheel"/>
+		<parent link="chassis"/>
+		<axis xyz="0 0 1" rpy="0 0 0"/>
+		<limit effort="10000" velocity="1000"/>
+		<joint_properties damping="1.0" friction="0.0"/>
+  	</joint>
+  	<joint type="continuous" name="right_front_wheel_hinge">
+		<origin xyz="0.06 -0.07 0" rpy="1.570796 0 0"/>
+		<child link="rightf_wheel"/>
+		<parent link="chassis"/>
+		<axis xyz="0 0 1" rpy="0 0 0"/>
+		<limit effort="10000" velocity="1000"/>
+		<joint_properties damping="1.0" friction="0.0"/>
+  	</joint>
 </robot>

File: urdfUdacityBot/besh udacity_bot.xacro (robot description, xacro)
@@ -1,4 +1,11 @@
 <?xml version='1.0'?>
 <robot name="udacity_bot" xmlns:xacro="http://www.ros.org/wiki/xacro">
+<xacro:include filename="$(find udacity_bot)/urdf/udacity_bot.gazebo" />
+  <link name="robot_footprint"></link>
+  <joint name="robot_footprint_joint" type="fixed">
+    <origin xyz="0 0 0" rpy="0 0 0" />
+    <parent link="robot_footprint"/>
+    <child link="chassis" />
+  </joint>
 	<link name='chassis'>
 		<inertial>
@@ -11,21 +18,21 @@
 		  />
 		</inertial>
-		<collision name='collision'>
+		<collision name='chassis_collision'>
 		  <origin xyz="0 0 0" rpy=" 0 0 0"/>
-		  <geometry>
-			<box size=".12 .14 .05"/>
-		  </geometry>
+     		 <geometry>
+     		   <box size=".24 .1 .02"/>
+    		  </geometry>
 		</collision>
 		<visual name='chassis_visual'>
 		  <origin xyz="0 0 0" rpy=" 0 0 0"/>
 		  <geometry>
-			<box size=".12 .14 .05"/>
+			<box size=".24 .1 .02"/>
 		  </geometry>
 		</visual>
 	</link>
 	<link name='rightb_wheel'>
-		<visual>
-			  <geometry>
-				<cylinder length="0.025" radius="0.03"/>
+		<visual >
+			  <geometry>
+				<cylinder length="0.025" radius="0.0335"/>
 			  </geometry>
 		</visual>
@@ -39,8 +46,8 @@
 			  />
     	</inertial>
-		<collision name='collision'>
-			  <origin xyz="0 0 0" rpy=" 0 0 0"/>
-			  <geometry>
-				<cylinder length="0.025" radius="0.03"/>
+		<collision>
+			  <origin xyz="0 0 0" rpy=" 0 0 0"/>
+			  <geometry>
+				<cylinder length="0.025" radius="0.0335"/>
 			  </geometry>
 			</collision>
@@ -49,5 +56,5 @@
 		<visual>
 			  <geometry>
-				<cylinder length="0.025" radius="0.03"/>
+				<cylinder length="0.025" radius="0.0335"/>
 			  </geometry>
 		</visual>
@@ -61,8 +68,8 @@
 			  />
     	</inertial>
-		<collision name='collision'>
-			  <origin xyz="0 0 0" rpy=" 0 0 0"/>
-			  <geometry>
-				<cylinder length="0.025" radius="0.03"/>
+		<collision>
+			  <origin xyz="0 0 0" rpy=" 0 0 0"/>
+			  <geometry>
+				<cylinder length="0.025" radius="0.0335"/>
 			  </geometry>
 			</collision>
@@ -71,5 +78,5 @@
 		<visual>
 			  <geometry>
-				<cylinder length="0.025" radius="0.03"/>
+				<cylinder length="0.025" radius="0.0335"/>
 			  </geometry>
 		</visual>
@@ -83,8 +90,8 @@
 			  />
     		</inertial>
-		<collision name='collision'>
-			  <origin xyz="0 0 0" rpy=" 0 0 0"/>
-			  <geometry>
-				<cylinder length="0.025" radius="0.03"/>
+		<collision>
+			  <origin xyz="0 0 0" rpy=" 0 0 0"/>
+			  <geometry>
+				<cylinder length="0.025" radius="0.0335"/>
 			  </geometry>
 			</collision>
@@ -93,76 +100,77 @@
 		<visual>
 			  <geometry>
+				<cylinder length="0.025" radius="0.0335"/>
+			  </geometry>
+		</visual>
+		<inertial>
+			  <mass value="0.033"/>
+			  <origin xyz="0.0 0 0" rpy=" 0 0 0"/>
+			  <inertia
+				  ixx="0.1" ixy="0" ixz="0"
+				  iyy="0.1" iyz="0"
+				  izz="0.1"
+			  />
+    	</inertial>
+		<collision>
+			  <origin xyz="0 0 0" rpy=" 0 0 0"/>
+			  <geometry>
 				<cylinder length="0.025" radius="0.03"/>
 			  </geometry>
-		</visual>
-		<inertial>
-			  <mass value="0.033"/>
-			  <origin xyz="0.0 0 0" rpy=" 0 0 0"/>
-			  <inertia
-				  ixx="0.1" ixy="0" ixz="0"
-				  iyy="0.1" iyz="0"
-				  izz="0.1"
-			  />
-    	</inertial>
-		<collision name='collision'>
-			  <origin xyz="0 0 0" rpy=" 0 0 0"/>
-			  <geometry>
-				<cylinder length="0.025" radius="0.03"/>
-			  </geometry>
-			</collision>
-	</link>
-	<link name='camera'>
-		<inertial>
-		  <mass value="0.050"/>
-		  <origin xyz="0.0 0 0" rpy=" 0 0 0"/>
-		  <inertia
-			  ixx="0.1" ixy="0" ixz="0"
-			  iyy="0.1" iyz="0"
-			  izz="0.1"
-		  />
-		</inertial>
-		<collision name='camera_collision'>
-		  <origin xyz="0 0 0" rpy=" 0 0 0"/>
-		  <geometry>
-			<box size=".005 .005 .005"/>
-		  </geometry>
-		</collision>
-		<visual name='camera_visual'>
-		  <origin xyz="0 0 0" rpy=" 0 0 0"/>
-		  <geometry>
-			<box size=".005 .005 .005"/>
-		  </geometry>
-		</visual>
-	</link>
-	<link name='range_finder'>
-		<inertial>
-		  <mass value="0.050"/>
-		  <origin xyz="0.0 0 0" rpy=" 0 0 0"/>
-		  <inertia
-			  ixx="0.1" ixy="0" ixz="0"
-			  iyy="0.1" iyz="0"
-			  izz="0.1"
-		  />
-		</inertial>
-		<collision name='range_finder_collision'>
-		  <origin xyz="0 0 0" rpy=" 0 0 0"/>
-		  <geometry>
-			<box size=".005 .005 .005"/>
-		  </geometry>
-		</collision>
-		<visual name='range_finder_visual'>
-		  <origin xyz="0 0 0" rpy=" 0 0 0"/>
-		<mesh filename="~/catkin_ws/src/udacity_bot/meshes/hokuyo.dae"/>
-		</visual>
-	</link>
+			</collision>
+	</link>
+	<link name="camera">
+     <visual>
+      <origin xyz="0 0 0" rpy="0 0 0"/>
+       <geometry>
+        <box size=".05 .05 .05"/>
+      </geometry>
+    </visual>
+    <inertial>
+      <mass value="0.1"/>
+      <origin xyz="0 0 0" rpy=" 0 0 0"/>
+      <inertia
+          ixx="0.000001" ixy="0" ixz="0"
+          iyy="0.000001" iyz="0"
+          izz="0.000001"
+      />
+    </inertial>
+    <collision>
+      <origin xyz="0 0 0" rpy="0 0 0"/>
+       <geometry>
+        <box size=".005 .005 .005"/>
+      </geometry>
+    </collision>
+</link>
+<link name="hokuyo">
+     <visual>
+      <origin xyz="0 0 0" rpy="0 0 0"/>
+       <geometry>
+	<mesh filename="package://udacity_bot/meshes/hokuyo.dae"/>
+      </geometry>
+    </visual>
+    <inertial>
+      <mass value="0.1"/>
+      <origin xyz="0 0 0" rpy=" 0 0 0"/>
+      <inertia
+          ixx="0.000001" ixy="0" ixz="0"
+          iyy="0.000001" iyz="0"
+          izz="0.000001"
+      />
+    </inertial>
+    <collision>
+      <origin xyz="0 0 0" rpy="0 0 0"/>
+       <geometry>
+        <box size=".05 .05 .05"/>
+      </geometry>
+    </collision>
+</link>
+  <joint name="hokuyo_joint" type="fixed">
+    <origin xyz="-0.005 0 0.127" rpy="0 0 0"/>
+    <parent link="chassis"/>
+    <child link="hokuyo"/>
+  </joint>
 	<joint type="fixed" name="camera_joint">
-		<origin xyz="0 0 0.027" rpy="0 0 0"/>
+		<origin xyz="0 0 0.119" rpy="0 0 0"/>
 		<child link="camera"/>
-		<parent link="chassis"/>
-		<axis xyz="0 0 0" rpy="0 0 0"/>
-  	</joint>
-	<joint type="fixed" name="range_finder_joint">
-		<origin xyz="-0.005 0 0.027" rpy="0 0 0"/>
-		<child link="range_finder"/>
 		<parent link="chassis"/>
 		<axis xyz="0 0 0" rpy="0 0 0"/>
