Commit message: Udacity robot able to reach goal

File: urdf/robot.urdf (robot description, URDF)
Before this commit: robot udacity_bot, 8 links, 7 joints
Links:
- removed link hokuyo
- removed link leftb_wheel
- removed link leftf_wheel
- removed link rightb_wheel
- removed link rightf_wheel
- added link left_wheel, mass 5.0; collision cylinder length=0.05 radius=0.1; visual cylinder length=0.05 radius=0.1
- added link right_wheel, mass 5.0; collision cylinder length=0.05 radius=0.1; visual cylinder length=0.05 radius=0.1
- link camera: geometry collision box size=0.05; visual box size=0.05
- link chassis: mass 0.489 -> 15.0; geometry collision box size=.4 .2 .1; collision sphere radius=0.05
Joints:
- removed joint hokuyo_joint
- removed joint left__back_wheel_hinge
- removed joint left__front_wheel_hinge
- removed joint right_back_wheel_hinge
- removed joint right_front_wheel_hinge
- added joint left_wheel_hinge: type continuous, parent chassis, child left_wheel, origin xyz=0 0.15 0 rpy=0 0 0, axis 0 1 0, limit effort=10000 velocity=1000
- added joint right_wheel_hinge: type continuous, parent chassis, child right_wheel, origin xyz=0 -0.15 0 rpy=0 0 0, axis 0 1 0, limit effort=10000 velocity=1000
- joint camera_joint: axis 0 0 0 -> (none); origin xyz=0 0 0.119 rpy=0 0 0 -> xyz=0.2 0.0 0 rpy=0 0 0; type fixed -> rigid

File: urdf/udacity_bot.xacro (robot description, xacro)
@@ -9,137 +9,136 @@
   </joint>
   <link name='chassis'>
-	<pose>0 0 0.1 0 0 0</pose>
-	<inertial>
-		<mass value="0.5"/>
-		<origin xyz="0.0 0 0" rpy=" 0 0 0"/>
-		<inertia
-			  ixx="0.1" ixy="0" ixz="0"
-			  iyy="0.1" iyz="0"
-			  izz="0.1"
-		/>
-	</inertial>
-	<collision name='chassis_collision'>
-		<origin xyz="0 0 0" rpy=" 0 0 0"/>
-     		<geometry>
-     			<box size=".24 .1 .02"/>
-    		</geometry>
-	</collision>
-	<visual name='chassis_visual'>
-		  <origin xyz="0 0 0" rpy=" 0 0 0"/>
-		  <geometry>
-			<box size=".24 .1 .02"/>
-		  </geometry>
-	</visual>
-		<visual name="rightb_wheel_visual" >
-		<origin xyz="-0.06 0.07 0" rpy="1.570796 0 0"/>
-			  <geometry>
-				<cylinder length="0.025" radius="0.0335"/>
-			  </geometry>
-		</visual>
-		<inertial>
-			  <mass value="0.033"/>
-			  <origin xyz="0.0 0 0" rpy=" 0 0 0"/>
-			  <inertia
-				  ixx="0.1" ixy="0" ixz="0"
-				  iyy="0.1" iyz="0"
-				  izz="0.1"
-			  />
-    	  	</inertial>
-		<collision name="rightb_wheel_collision">
-			<origin xyz="-0.06 0.07 0" rpy="1.570796 0 0"/>
-			  <geometry>
-				<cylinder length="0.025" radius="0.0335"/>
-			  </geometry>
-		 <surface>
-        		<friction>
-         		 <ode>
-         		   <mu>0</mu>
-          		  <mu2>0</mu2>
-           		 <slip1>1.0</slip1>
-          		  <slip2>1.0</slip2>
-         			 </ode>
-       			 </friction>
+    <pose>0 0 0.1 0 0 0</pose>
+    <inertial>
+      <mass value="15"/>
+      <origin xyz="0.0 0 0" rpy=" 0 0 0"/>
+      <inertia
+          ixx="0.1" ixy="0" ixz="0"
+          iyy="0.1" iyz="0"
+          izz="0.1"
+      />
+    </inertial>
+    <collision name='collision'>
+      <origin xyz="0 0 0" rpy=" 0 0 0"/>
+      <geometry>
+        <box size=".4 .2 .1"/>
+      </geometry>
+    </collision>
+    <visual name='chassis_visual'>
+     <origin xyz="0 0 0" rpy=" 0 0 0"/>
+      <geometry>
+        <box size=".4 .2 .1"/>
+      </geometry>
+    </visual>
+    <visual name='back_caster_visual'>
+      <origin xyz="-0.15 0 -0.05" rpy=" 0 0 0"/>
+      <geometry>
+        <sphere radius="0.0499"/>
+      </geometry>
+    </visual>
+    <collision name='back_caster_collision'>
+	<origin xyz="-0.15 0 -0.05" rpy=" 0 0 0"/>
+      	<geometry>
+          <sphere radius="0.0499"/>
+      	</geometry>
+      <surface>
+        <friction>
+          <ode>
+            <mu>0</mu>
+            <mu2>0</mu2>
+            <slip1>1.0</slip1>
+            <slip2>1.0</slip2>
+          </ode>
+        </friction>
       </surface>
-		</collision>
-		<visual name="leftb_wheel_visual">
-		<origin xyz="-0.06 -0.07 0" rpy="1.570796 0 0"/>
-			  <geometry>
-				<cylinder length="0.025" radius="0.0335"/>
-			  </geometry>
-		</visual>
-		<inertial>
-			  <mass value="0.033"/>
-			  <origin xyz="0.0 0 0" rpy=" 0 0 0"/>
-			  <inertia
-				  ixx="0.1" ixy="0" ixz="0"
-				  iyy="0.1" iyz="0"
-				  izz="0.1"
-			  />
-    		</inertial>
-		<collision name="leftb_wheel_collision">
-		<origin xyz="-0.06 -0.07 0" rpy="1.570796 0 0"/>
-			  <geometry>
-				<cylinder length="0.025" radius="0.0335"/>
-			  </geometry>
- 			<surface>
-        		 <friction>
-         		 	<ode>
-         		 	  <mu>0</mu>
-          		 	 <mu2>0</mu2>
-           			 <slip1>1.0</slip1>
-          			  <slip2>1.0</slip2>
-         			 </ode>
-       			 </friction>
-      			</surface>
-		</collision>
+    </collision>
+    <collision name='front_caster_collision'>
+      <origin xyz="0.15 0 -0.05" rpy=" 0 0 0"/>
+      <geometry>
+        <sphere radius="0.0499"/>
+      </geometry>
+      <surface>
+        <friction>
+          <ode>
+            <mu>0</mu>
+            <mu2>0</mu2>
+            <slip1>1.0</slip1>
+            <slip2>1.0</slip2>
+          </ode>
+        </friction>
+      </surface>
+    </collision>
+    <visual name='front_caster_visual'>
+      <origin xyz="0.15 0 -0.05" rpy=" 0 0 0"/>
+      <geometry>
+        <sphere radius="0.0499"/>
+      </geometry>
+    </visual>
   </link>
-	<link name='rightf_wheel'>
-		<visual>
-		 <origin xyz="0.0 0 0" rpy=" 0 0 0"/>
-			  <geometry>
-				<cylinder length="0.025" radius="0.0335"/>
-			  </geometry>
-		</visual>
-		<inertial>
-			  <mass value="0.033"/>
-			  <origin xyz="0.0 0 0" rpy=" 0 0 0"/>
-			  <inertia
-				  ixx="0.1" ixy="0" ixz="0"
-				  iyy="0.1" iyz="0"
-				  izz="0.1"
-			  />
-    		</inertial>
-		<collision>
-		<origin xyz="0.0 0 0" rpy=" 0 0 0"/>
-			  <geometry>
-				<cylinder length="0.025" radius="0.0335"/>
-			  </geometry>
-			</collision>
-	</link>
-	<link name='leftf_wheel'>
-		<visual>
-			  <geometry>
-				<cylinder length="0.025" radius="0.0335"/>
-			  </geometry>
-		</visual>
-		<inertial>
-			  <mass value="0.033"/>
-			  <origin xyz="0.0 0 0" rpy=" 0 0 0"/>
-			  <inertia
-				  ixx="0.1" ixy="0" ixz="0"
-				  iyy="0.1" iyz="0"
-				  izz="0.1"
-			  />
-    		</inertial>
-		<collision>
-			  <origin xyz="0 0 0" rpy=" 0 0 0"/>
-			  <geometry>
-				<cylinder length="0.025" radius="0.03"/>
-			  </geometry>
-		</collision>
-	</link>
-	<link name="camera">
+  <link name="right_wheel">
+    <visual>
+      <origin xyz="0 0 0" rpy="0 1.5707 1.5707"/>
+       <geometry>
+        <cylinder length="0.05" radius="0.1"/>
+      </geometry>
+    </visual>
+    <inertial>
+      <mass value="5"/>
+      <origin xyz="0.0 0 0" rpy=" 0 0 0"/>
+      <inertia
+          ixx="0.1" ixy="0" ixz="0"
+          iyy="0.1" iyz="0"
+          izz="0.1"
+      />
+    </inertial>
+	<collision>
+      <origin xyz="0 0 0" rpy="0 1.5707 1.5707"/>
+       <geometry>
+        <cylinder length="0.05" radius="0.1"/>
+      </geometry>
+    </collision>
+ </link>
+  <link name="left_wheel">
+    <visual>
+      <origin xyz="0 0 0" rpy="0 1.5707 1.5707"/>
+       <geometry>
+        <cylinder length="0.05" radius="0.1"/>
+      </geometry>
+    </visual>
+    <inertial>
+      <mass value="5"/>
+      <origin xyz="0.0 0 0" rpy=" 0 0 0"/>
+      <inertia
+          ixx="0.1" ixy="0" ixz="0"
+          iyy="0.1" iyz="0"
+          izz="0.1"
+      />
+    </inertial>
+	<collision>
+      <origin xyz="0 0 0" rpy="0 1.5707 1.5707"/>
+       <geometry>
+        <cylinder length="0.05" radius="0.1"/>
+      </geometry>
+    </collision>
+  </link>
+<joint type="continuous" name="left_wheel_hinge">
+    <origin xyz="0 0.15 0" rpy="0 0 0"/>
+    <child link="left_wheel"/>
+    <parent link="chassis"/>
+    <axis xyz="0 1 0" rpy="0 0 0"/>
+    <limit effort="10000" velocity="1000"/>
+    <joint_properties damping="1.0" friction="1.0"/>
+  </joint>
+<joint type="continuous" name="right_wheel_hinge">
+    <origin xyz="0 -0.15 0" rpy="0 0 0"/>
+    <child link="right_wheel"/>
+    <parent link="chassis"/>
+    <axis xyz="0 1 0" rpy="0 0 0"/>
+    <limit effort="10000" velocity="1000"/>
+    <joint_properties damping="1.0" friction="1.0"/>
+  </joint>
+<link name="camera">
      <visual>
-     	<origin xyz="0 0 0" rpy="0 0 0"/>
+      <origin xyz="0 0 0" rpy="0 0 0"/>
        <geometry>
         <box size=".05 .05 .05"/>
@@ -147,5 +146,5 @@
     </visual>
     <inertial>
-      <mass value="0.01"/>
+      <mass value="0.1"/>
       <origin xyz="0 0 0" rpy=" 0 0 0"/>
       <inertia
@@ -162,4 +161,9 @@
     </collision>
 </link>
+  <joint name="camera_robot_joint" type="fixed">
+    <origin xyz="0.2 0 0" rpy="0 0 0" />
+    <parent link="chassis"/>
+    <child link="camera"/>
+  </joint>
 <link name="hokuyo">
      <visual>
@@ -178,37 +182,15 @@
       />
     </inertial>
-	    <collision>
-	      <origin xyz="0 0 0" rpy="0 0 0"/>
-	       <geometry>
-	        <box size=".05 .05 .05"/>
-	      </geometry>
-	    </collision>
-	</link>
-	  <joint name="hokuyo_joint" type="fixed">
-	    <origin xyz="0.13 0 0.127" rpy="0 0 0"/>
-	    <parent link="chassis"/>
-	    <child link="hokuyo"/>
-	  </joint>
-	<joint type="fixed" name="camera_joint">
-		<origin xyz="0.13 0.05 0.07" rpy="0 0 0"/>
-		<child link="camera"/>
-		<parent link="chassis"/>
-		<axis xyz="0 0 0" rpy="0 0 0"/>
-  	</joint>
-	<joint type="continuous" name="left__front_wheel_hinge">
-		<origin xyz="0.06 0.07 0" rpy="1.570796 0 0"/>
-		<child link="leftf_wheel"/>
-		<parent link="chassis"/>
-		<axis xyz="0 0 1" rpy="0 0 0"/>
-		<limit effort="10000" velocity="1000"/>
-		<joint_properties damping="1.0" friction="0.0"/>
-  	</joint>
-  	<joint type="continuous" name="right_front_wheel_hinge">
-		<origin xyz="0.06 -0.07 0" rpy="1.570796 0 0"/>
-		<child link="rightf_wheel"/>
-		<parent link="chassis"/>
-		<axis xyz="0 0 1" rpy="0 0 0"/>
-		<limit effort="10000" velocity="1000"/>
-		<joint_properties damping="1.0" friction="0.0"/>
-  	</joint>
+    <collision>
+      <origin xyz="0 0 0" rpy="0 0 0"/>
+       <geometry>
+        <box size=".05 .05 .05"/>
+      </geometry>
+    </collision>
+</link>
+  <joint name="hokuyo_joint" type="fixed">
+    <origin xyz=".15 0 .1 " rpy="0 0 0" />
+    <parent link="chassis"/>
+    <child link="hokuyo"/>
+  </joint>
 </robot>

File: urdfCircleBot/udacity_bot.xacro (robot description, xacro)
@@ -9,8 +9,8 @@
   </joint>
   <link name='chassis'>
-    <pose>0 0 0.1 0 0 0</pose>
+    <pose>0 0 0.2 0 0 0</pose>
     <inertial>
-      <mass value="0.3"/>
-      <origin xyz="0.0 0 0" rpy=" 0 0 0"/>
+      <mass value="15.0"/>
+      <origin xyz="0.05 0 0" rpy=" 0 0 0"/>
       <inertia
           ixx="0.1" ixy="0" ixz="0"
@@ -19,8 +19,8 @@
       />
     </inertial>
-    <collision name='collision'>
+    <collision name='chassis_collision'>
       <origin xyz="0 0 0" rpy=" 0 0 0"/>
       <geometry>
-        <box size=".24 0.1 .02"/>
+	<cylinder length="0.05" radius="0.15"/>
       </geometry>
     </collision>
@@ -28,18 +28,12 @@
      <origin xyz="0 0 0" rpy=" 0 0 0"/>
       <geometry>
-        <box size=".4 .2 .1"/>
-      </geometry>
-    </visual>
-    <visual name='back_caster_visual'>
-      <origin xyz="-0.15 0 -0.05" rpy=" 0 0 0"/>
-      <geometry>
-        <sphere radius="0.05"/>
+	<cylinder length="0.05" radius="0.15"/>
       </geometry>
     </visual>
     <collision name='back_caster_collision'>
-	<origin xyz="-0.15 0 -0.05" rpy=" 0 0 0"/>
-      	<geometry>
-          <sphere radius="0.0499"/>
-      	</geometry>
+     <origin xyz="-0.1 0 0.0" rpy=" 0 0 0"/>
+      <geometry>
+        <sphere radius="0.0499"/>
+      </geometry>
       <surface>
         <friction>
@@ -53,6 +47,12 @@
       </surface>
     </collision>
+    <visual name='back_caster_visual'>
+     <origin xyz="-0.1 0 -0.0" rpy=" 0 0 0"/>
+      <geometry>
+        <sphere radius="0.0499"/>
+      </geometry>
+    </visual>
     <collision name='front_caster_collision'>
-      <origin xyz="0.15 0 -0.05" rpy=" 0 0 0"/>
+     <origin xyz="0.1 0 0.0" rpy=" 0 0 0"/>
       <geometry>
         <sphere radius="0.0499"/>
@@ -70,7 +70,7 @@
     </collision>
     <visual name='front_caster_visual'>
-      <origin xyz="0.15 0 -0.05" rpy=" 0 0 0"/>
+     <origin xyz="0.1 0 0.0" rpy=" 0 0 0"/>
       <geometry>
-        <sphere radius="0.05"/>
+        <sphere radius="0.04999"/>
       </geometry>
     </visual>
@@ -80,9 +80,9 @@
       <origin xyz="0 0 0" rpy="0 1.5707 1.5707"/>
        <geometry>
-        <cylinder length="0.05" radius="0.1"/>
+        <cylinder length="0.025" radius="0.05"/>
       </geometry>
     </visual>
     <inertial>
-      <mass value="0.5"/>
+      <mass value="5"/>
       <origin xyz="0.0 0 0" rpy=" 0 0 0"/>
       <inertia
@@ -95,5 +95,5 @@
       <origin xyz="0 0 0" rpy="0 1.5707 1.5707"/>
        <geometry>
-        <cylinder length="0.05" radius="0.1"/>
+        <cylinder length="0.025" radius="0.05"/>
       </geometry>
     </collision>
@@ -103,9 +103,9 @@
       <origin xyz="0 0 0" rpy="0 1.5707 1.5707"/>
        <geometry>
-        <cylinder length="0.05" radius="0.1"/>
+        <cylinder length="0.025" radius="0.05"/>
       </geometry>
     </visual>
     <inertial>
-      <mass value="0.5"/>
+      <mass value="5"/>
       <origin xyz="0.0 0 0" rpy=" 0 0 0"/>
       <inertia
@@ -118,10 +118,10 @@
       <origin xyz="0 0 0" rpy="0 1.5707 1.5707"/>
        <geometry>
-        <cylinder length="0.05" radius="0.1"/>
+        <cylinder length="0.025" radius="0.05"/>
       </geometry>
     </collision>
   </link>
 <joint type="continuous" name="left_wheel_hinge">
-    <origin xyz="0 0.15 0" rpy="0 0 0"/>
+    <origin xyz="0 0.175 0" rpy="0 0 0"/>
     <child link="left_wheel"/>
     <parent link="chassis"/>
@@ -131,5 +131,5 @@
   </joint>
 <joint type="continuous" name="right_wheel_hinge">
-    <origin xyz="0 -0.15 0" rpy="0 0 0"/>
+    <origin xyz="0 -0.175 0" rpy="0 0 0"/>
     <child link="right_wheel"/>
     <parent link="chassis"/>
@@ -162,5 +162,5 @@
 </link>
   <joint name="camera_robot_joint" type="fixed">
-    <origin xyz="0.2 0 0" rpy="0 0 0" />
+    <origin xyz="0.1 0 0.1" rpy="0 0 0" />
     <parent link="chassis"/>
     <child link="camera"/>
@@ -190,5 +190,5 @@
 </link>
   <joint name="hokuyo_joint" type="fixed">
-    <origin xyz=".15 0 .1 " rpy="0 0 0" />
+    <origin xyz=".1 0 .16 " rpy="0 0 0" />
     <parent link="chassis"/>
     <child link="hokuyo"/>
