Commit message: sample bot goal reached

File: urdf/udacity_bot.xacro (robot description, xacro)
@@ -1,146 +1,196 @@
 <?xml version='1.0'?>
 <robot name="udacity_bot" xmlns:xacro="http://www.ros.org/wiki/xacro">
-	<link name='chassis'>
-		<inertial>
-		  <mass value="0.489"/>
-		  <origin xyz="0.0 0 0" rpy=" 0 0 0"/>
-		  <inertia
-			  ixx="0.1" ixy="0" ixz="0"
-			  iyy="0.1" iyz="0"
-			  izz="0.1"
-		  />
-		</inertial>
-		<collision name='collision'>
-		  <origin xyz="0 0 0" rpy=" 0 0 0"/>
-		  <geometry>
-			<box size=".12 .14 .05"/>
-		  </geometry>
-		</collision>
-		<visual name='chassis_visual'>
-		  <origin xyz="0 0 0" rpy=" 0 0 0"/>
-		  <geometry>
-			<box size=".12 .14 .05"/>
-		  </geometry>
-		</visual>
-	</link>
-	<link name='rightb_wheel'>
-		<visual>
-			  <geometry>
-				<cylinder length="0.025" radius="0.03"/>
-			  </geometry>
-		</visual>
-		<inertial>
-			  <mass value="0.033"/>
-			  <origin xyz="0.0 0 0" rpy=" 0 0 0"/>
-			  <inertia
-				  ixx="0.1" ixy="0" ixz="0"
-				  iyy="0.1" iyz="0"
-				  izz="0.1"
-			  />
-    	</inertial>
-		<collision name='collision'>
-			  <origin xyz="0 0 0" rpy=" 0 0 0"/>
-			  <geometry>
-				<cylinder length="0.025" radius="0.03"/>
-			  </geometry>
-			</collision>
-	</link>
-	<link name='leftb_wheel'>
-		<visual>
-			  <geometry>
-				<cylinder length="0.025" radius="0.03"/>
-			  </geometry>
-		</visual>
-		<inertial>
-			  <mass value="0.033"/>
-			  <origin xyz="0.0 0 0" rpy=" 0 0 0"/>
-			  <inertia
-				  ixx="0.1" ixy="0" ixz="0"
-				  iyy="0.1" iyz="0"
-				  izz="0.1"
-			  />
-    	</inertial>
-		<collision name='collision'>
-			  <origin xyz="0 0 0" rpy=" 0 0 0"/>
-			  <geometry>
-				<cylinder length="0.025" radius="0.03"/>
-			  </geometry>
-			</collision>
-	</link>
-	<link name='rightf_wheel'>
-		<visual>
-			  <geometry>
-				<cylinder length="0.025" radius="0.03"/>
-			  </geometry>
-		</visual>
-		<inertial>
-			  <mass value="0.033"/>
-			  <origin xyz="0.0 0 0" rpy=" 0 0 0"/>
-			  <inertia
-				  ixx="0.1" ixy="0" ixz="0"
-				  iyy="0.1" iyz="0"
-				  izz="0.1"
-			  />
-    		</inertial>
-		<collision name='collision'>
-			  <origin xyz="0 0 0" rpy=" 0 0 0"/>
-			  <geometry>
-				<cylinder length="0.025" radius="0.03"/>
-			  </geometry>
-			</collision>
-	</link>
-	<link name='leftf_wheel'>
-		<visual>
-			  <geometry>
-				<cylinder length="0.025" radius="0.03"/>
-			  </geometry>
-		</visual>
-		<inertial>
-			  <mass value="0.033"/>
-			  <origin xyz="0.0 0 0" rpy=" 0 0 0"/>
-			  <inertia
-				  ixx="0.1" ixy="0" ixz="0"
-				  iyy="0.1" iyz="0"
-				  izz="0.1"
-			  />
-    	</inertial>
-		<collision name='collision'>
-			  <origin xyz="0 0 0" rpy=" 0 0 0"/>
-			  <geometry>
-				<cylinder length="0.025" radius="0.03"/>
-			  </geometry>
-			</collision>
-	</link>
-	<joint type="continuous" name="left__back_wheel_hinge">
-		<origin xyz="0.06 -0.07 0" rpy="1.570796 0 0"/>
-		<child link="leftb_wheel"/>
-		<parent link="chassis"/>
-		<axis xyz="0 1 0" rpy="0 0 0"/>
-		<limit effort="10000" velocity="1000"/>
-		<joint_properties damping="1.0" friction="1.0"/>
-  	</joint>
-  	<joint type="continuous" name="right_back_wheel_hinge">
-		<origin xyz="0.06 0.07 0" rpy="1.570796 0 0"/>
-		<child link="rightb_wheel"/>
-		<parent link="chassis"/>
-		<axis xyz="0 1 0" rpy="0 0 0"/>
-		<limit effort="10000" velocity="1000"/>
-		<joint_properties damping="1.0" friction="1.0"/>
-  	</joint>
-	<joint type="continuous" name="left__front_wheel_hinge">
-		<origin xyz="-0.06 -0.07 0" rpy="1.570796 0 0"/>
-		<child link="leftf_wheel"/>
-		<parent link="chassis"/>
-		<axis xyz="0 1 0" rpy="0 0 0"/>
-		<limit effort="10000" velocity="1000"/>
-		<joint_properties damping="1.0" friction="1.0"/>
-  	</joint>
-  	<joint type="continuous" name="right_front_wheel_hinge">
-		<origin xyz="-0.06 0.07 0" rpy="1.570796 0 0"/>
-		<child link="rightf_wheel"/>
-		<parent link="chassis"/>
-		<axis xyz="0 1 0" rpy="0 0 0"/>
-		<limit effort="10000" velocity="1000"/>
-		<joint_properties damping="1.0" friction="1.0"/>
-  	</joint>
+<xacro:include filename="$(find udacity_bot)/urdf/udacity_bot.gazebo" />
+  <link name="robot_footprint"></link>
+  <joint name="robot_footprint_joint" type="fixed">
+    <origin xyz="0 0 0" rpy="0 0 0" />
+    <parent link="robot_footprint"/>
+    <child link="chassis" />
+  </joint>
+  <link name='chassis'>
+    <pose>0 0 0.1 0 0 0</pose>
+    <inertial>
+      <mass value="15.0"/>
+      <origin xyz="0.0 0 0" rpy=" 0 0 0"/>
+      <inertia
+          ixx="0.1" ixy="0" ixz="0"
+          iyy="0.1" iyz="0"
+          izz="0.1"
+      />
+    </inertial>
+    <collision name='collision'>
+      <origin xyz="0 0 0" rpy=" 0 0 0"/>
+      <geometry>
+        <box size=".4 .2 .1"/>
+      </geometry>
+    </collision>
+    <visual name='chassis_visual'>
+      <origin xyz="0 0 0" rpy=" 0 0 0"/>
+      <geometry>
+        <box size=".4 .2 .1"/>
+      </geometry>
+    </visual>
+    <visual name='back_caster_visual'>
+      <origin xyz="-0.15 0 -0.05" rpy=" 0 0 0"/>
+      <geometry>
+        <sphere radius="0.05"/>
+      </geometry>
+    </visual>
+    <collision name='back_caster_collision'>
+	<origin xyz="-0.15 0 -0.05" rpy=" 0 0 0"/>
+      	<geometry>
+          <sphere radius="0.0499"/>
+      	</geometry>
+      <surface>
+        <friction>
+          <ode>
+            <mu>0</mu>
+            <mu2>0</mu2>
+            <slip1>1.0</slip1>
+            <slip2>1.0</slip2>
+          </ode>
+        </friction>
+      </surface>
+    </collision>
+    <collision name='front_caster_collision'>
+      <origin xyz="0.15 0 -0.05" rpy=" 0 0 0"/>
+      <geometry>
+        <sphere radius="0.0499"/>
+      </geometry>
+      <surface>
+        <friction>
+          <ode>
+            <mu>0</mu>
+            <mu2>0</mu2>
+            <slip1>1.0</slip1>
+            <slip2>1.0</slip2>
+          </ode>
+        </friction>
+      </surface>
+    </collision>
+    <visual name='front_caster_visual'>
+      <origin xyz="0.15 0 -0.05" rpy=" 0 0 0"/>
+      <geometry>
+        <sphere radius="0.05"/>
+      </geometry>
+    </visual>
+  </link>
+  <link name="right_wheel">
+    <visual>
+      <origin xyz="0 0 0" rpy="0 1.5707 1.5707"/>
+       <geometry>
+        <cylinder length="0.05" radius="0.1"/>
+      </geometry>
+    </visual>
+    <inertial>
+      <mass value="5.0"/>
+      <origin xyz="0.0 0 0" rpy=" 0 0 0"/>
+      <inertia
+          ixx="0.1" ixy="0" ixz="0"
+          iyy="0.1" iyz="0"
+          izz="0.1"
+      />
+    </inertial>
+	<collision>
+      <origin xyz="0 0 0" rpy="0 1.5707 1.5707"/>
+       <geometry>
+        <cylinder length="0.05" radius="0.1"/>
+      </geometry>
+    </collision>
+ </link>
+  <link name="left_wheel">
+    <visual>
+      <origin xyz="0 0 0" rpy="0 1.5707 1.5707"/>
+       <geometry>
+        <cylinder length="0.05" radius="0.1"/>
+      </geometry>
+    </visual>
+    <inertial>
+      <mass value="5.0"/>
+      <origin xyz="0.0 0 0" rpy=" 0 0 0"/>
+      <inertia
+          ixx="0.1" ixy="0" ixz="0"
+          iyy="0.1" iyz="0"
+          izz="0.1"
+      />
+    </inertial>
+	<collision>
+      <origin xyz="0 0 0" rpy="0 1.5707 1.5707"/>
+       <geometry>
+        <cylinder length="0.05" radius="0.1"/>
+      </geometry>
+    </collision>
+  </link>
+<joint type="continuous" name="left_wheel_hinge">
+    <origin xyz="0 0.15 0" rpy="0 0 0"/>
+    <child link="left_wheel"/>
+    <parent link="chassis"/>
+    <axis xyz="0 1 0" rpy="0 0 0"/>
+    <limit effort="10000" velocity="1000"/>
+    <joint_properties damping="1.0" friction="1.0"/>
+  </joint>
+<joint type="continuous" name="right_wheel_hinge">
+    <origin xyz="0 -0.15 0" rpy="0 0 0"/>
+    <child link="right_wheel"/>
+    <parent link="chassis"/>
+    <axis xyz="0 1 0" rpy="0 0 0"/>
+    <limit effort="10000" velocity="1000"/>
+    <joint_properties damping="1.0" friction="1.0"/>
+  </joint>
+<link name="camera">
+     <visual>
+      <origin xyz="0 0 0" rpy="0 0 0"/>
+       <geometry>
+        <box size=".05 .05 .05"/>
+      </geometry>
+    </visual>
+    <inertial>
+      <mass value="0.1"/>
+      <origin xyz="0 0 0" rpy=" 0 0 0"/>
+      <inertia
+          ixx="0.000001" ixy="0" ixz="0"
+          iyy="0.000001" iyz="0"
+          izz="0.000001"
+      />
+    </inertial>
+    <collision>
+      <origin xyz="0 0 0" rpy="0 0 0"/>
+       <geometry>
+        <box size=".05 .05 .05"/>
+      </geometry>
+    </collision>
+</link>
+  <joint name="camera_robot_joint" type="fixed">
+    <origin xyz="0.2 0 0" rpy="0 0 0" />
+    <parent link="chassis"/>
+    <child link="camera"/>
+  </joint>
+<link name="hokuyo">
+     <visual>
+      <origin xyz="0 0 0" rpy="0 0 0"/>
+       <geometry>
+	<mesh filename="package://udacity_bot/meshes/hokuyo.dae"/>
+      </geometry>
+    </visual>
+    <inertial>
+      <mass value="0.1"/>
+      <origin xyz="0 0 0" rpy=" 0 0 0"/>
+      <inertia
+          ixx="0.000001" ixy="0" ixz="0"
+          iyy="0.000001" iyz="0"
+          izz="0.000001"
+      />
+    </inertial>
+    <collision>
+      <origin xyz="0 0 0" rpy="0 0 0"/>
+       <geometry>
+        <box size=".05 .05 .05"/>
+      </geometry>
+    </collision>
+</link>
+  <joint name="hokuyo_joint" type="fixed">
+    <origin xyz=".15 0 .1 " rpy="0 0 0" />
+    <parent link="chassis"/>
+    <child link="hokuyo"/>
+  </joint>
 </robot>

Commit message: ProjectFinished

File: urdf/udacity_bot.xacro (robot description, xacro)
@@ -9,8 +9,8 @@
   </joint>
   <link name='chassis'>
-    <pose>0 0 0.1 0 0 0</pose>
+    <pose>0 0 0.2 0 0 0</pose>
     <inertial>
-      <mass value="15"/>
-      <origin xyz="0.0 0 0" rpy=" 0 0 0"/>
+      <mass value="10.0"/>
+      <origin xyz="0.03 0 0" rpy=" 0 0 0"/>
       <inertia
           ixx="0.1" ixy="0" ixz="0"
@@ -19,8 +19,8 @@
       />
     </inertial>
-    <collision name='collision'>
+    <collision name='chassis_collision'>
       <origin xyz="0 0 0" rpy=" 0 0 0"/>
       <geometry>
-        <box size=".4 .2 .1"/>
+	<cylinder length="0.03" radius="0.2"/>
       </geometry>
     </collision>
@@ -28,18 +28,12 @@
      <origin xyz="0 0 0" rpy=" 0 0 0"/>
       <geometry>
-        <box size=".4 .2 .1"/>
-      </geometry>
-    </visual>
-    <visual name='back_caster_visual'>
-      <origin xyz="-0.15 0 -0.05" rpy=" 0 0 0"/>
-      <geometry>
-        <sphere radius="0.0499"/>
+	<cylinder length="0.03" radius="0.2"/>
       </geometry>
     </visual>
     <collision name='back_caster_collision'>
-	<origin xyz="-0.15 0 -0.05" rpy=" 0 0 0"/>
-      	<geometry>
-          <sphere radius="0.0499"/>
-      	</geometry>
+     <origin xyz="-0.2 0 -0.02" rpy=" 0 0 0"/>
+      <geometry>
+        <sphere radius="0.0399"/>
+      </geometry>
       <surface>
         <friction>
@@ -53,8 +47,14 @@
       </surface>
     </collision>
+    <visual name='back_caster_visual'>
+     <origin xyz="-0.2 0 -0.02" rpy=" 0 0 0"/>
+      <geometry>
+        <sphere radius="0.0399"/>
+      </geometry>
+    </visual>
     <collision name='front_caster_collision'>
-      <origin xyz="0.15 0 -0.05" rpy=" 0 0 0"/>
+     <origin xyz="0.2 0 -0.02" rpy=" 0 0 0"/>
       <geometry>
-        <sphere radius="0.0499"/>
+        <sphere radius="0.0399"/>
       </geometry>
       <surface>
@@ -70,7 +70,7 @@
     </collision>
     <visual name='front_caster_visual'>
-      <origin xyz="0.15 0 -0.05" rpy=" 0 0 0"/>
+     <origin xyz="0.2 0 -0.02" rpy=" 0 0 0"/>
       <geometry>
-        <sphere radius="0.0499"/>
+        <sphere radius="0.0399"/>
       </geometry>
     </visual>
@@ -80,9 +80,9 @@
       <origin xyz="0 0 0" rpy="0 1.5707 1.5707"/>
        <geometry>
-        <cylinder length="0.05" radius="0.1"/>
+        <cylinder length="0.025" radius="0.06"/>
       </geometry>
     </visual>
     <inertial>
-      <mass value="5"/>
+      <mass value="3"/>
       <origin xyz="0.0 0 0" rpy=" 0 0 0"/>
       <inertia
@@ -95,5 +95,5 @@
       <origin xyz="0 0 0" rpy="0 1.5707 1.5707"/>
        <geometry>
-        <cylinder length="0.05" radius="0.1"/>
+        <cylinder length="0.025" radius="0.06"/>
       </geometry>
     </collision>
@@ -103,9 +103,9 @@
       <origin xyz="0 0 0" rpy="0 1.5707 1.5707"/>
        <geometry>
-        <cylinder length="0.05" radius="0.1"/>
+        <cylinder length="0.025" radius="0.06"/>
       </geometry>
     </visual>
     <inertial>
-      <mass value="5"/>
+      <mass value="3"/>
       <origin xyz="0.0 0 0" rpy=" 0 0 0"/>
       <inertia
@@ -118,10 +118,10 @@
       <origin xyz="0 0 0" rpy="0 1.5707 1.5707"/>
        <geometry>
-        <cylinder length="0.05" radius="0.1"/>
+        <cylinder length="0.025" radius="0.06"/>
       </geometry>
     </collision>
   </link>
 <joint type="continuous" name="left_wheel_hinge">
-    <origin xyz="0 0.15 0" rpy="0 0 0"/>
+    <origin xyz="0 0.226 0" rpy="0 0 0"/>
     <child link="left_wheel"/>
     <parent link="chassis"/>
@@ -131,5 +131,5 @@
   </joint>
 <joint type="continuous" name="right_wheel_hinge">
-    <origin xyz="0 -0.15 0" rpy="0 0 0"/>
+    <origin xyz="0 -0.226 0" rpy="0 0 0"/>
     <child link="right_wheel"/>
     <parent link="chassis"/>
@@ -162,5 +162,5 @@
 </link>
   <joint name="camera_robot_joint" type="fixed">
-    <origin xyz="0.2 0 0" rpy="0 0 0" />
+    <origin xyz="0.1 0 0.1" rpy="0 0 0" />
     <parent link="chassis"/>
     <child link="camera"/>
@@ -190,5 +190,5 @@
 </link>
   <joint name="hokuyo_joint" type="fixed">
-    <origin xyz=".15 0 .1 " rpy="0 0 0" />
+    <origin xyz=".1 0 .16 " rpy="0 0 0" />
     <parent link="chassis"/>
     <child link="hokuyo"/>

File: urdfUdacityBot/udacity_bot.xacro (robot description, xacro)
@@ -9,8 +9,8 @@
   </joint>
   <link name='chassis'>
-    <pose>0 0 0.2 0 0 0</pose>
+    <pose>0 0 0.1 0 0 0</pose>
     <inertial>
-      <mass value="10.0"/>
-      <origin xyz="0.03 0 0" rpy=" 0 0 0"/>
+      <mass value="15"/>
+      <origin xyz="0.0 0 0" rpy=" 0 0 0"/>
       <inertia
           ixx="0.1" ixy="0" ixz="0"
@@ -19,8 +19,8 @@
       />
     </inertial>
-    <collision name='chassis_collision'>
+    <collision name='collision'>
       <origin xyz="0 0 0" rpy=" 0 0 0"/>
       <geometry>
-	<cylinder length="0.05" radius="0.25"/>
+        <box size=".4 .2 .1"/>
       </geometry>
     </collision>
@@ -28,12 +28,18 @@
      <origin xyz="0 0 0" rpy=" 0 0 0"/>
       <geometry>
-	<cylinder length="0.05" radius="0.25"/>
+        <box size=".4 .2 .1"/>
+      </geometry>
+    </visual>
+    <visual name='back_caster_visual'>
+      <origin xyz="-0.15 0 -0.05" rpy=" 0 0 0"/>
+      <geometry>
+        <sphere radius="0.0499"/>
       </geometry>
     </visual>
     <collision name='back_caster_collision'>
-     <origin xyz="-0.24 0 -0.02" rpy=" 0 0 0"/>
-      <geometry>
-        <sphere radius="0.0299"/>
-      </geometry>
+	<origin xyz="-0.15 0 -0.05" rpy=" 0 0 0"/>
+      	<geometry>
+          <sphere radius="0.0499"/>
+      	</geometry>
       <surface>
         <friction>
@@ -47,14 +53,8 @@
       </surface>
     </collision>
-    <visual name='back_caster_visual'>
-     <origin xyz="-0.24 0 -0.02" rpy=" 0 0 0"/>
+    <collision name='front_caster_collision'>
+      <origin xyz="0.15 0 -0.05" rpy=" 0 0 0"/>
       <geometry>
-        <sphere radius="0.0299"/>
-      </geometry>
-    </visual>
-    <collision name='front_caster_collision'>
-     <origin xyz="0.2 0 -0.02" rpy=" 0 0 0"/>
-      <geometry>
-        <sphere radius="0.0299"/>
+        <sphere radius="0.0499"/>
       </geometry>
       <surface>
@@ -70,7 +70,7 @@
     </collision>
     <visual name='front_caster_visual'>
-     <origin xyz="0.2 0 -0.02" rpy=" 0 0 0"/>
+      <origin xyz="0.15 0 -0.05" rpy=" 0 0 0"/>
       <geometry>
-        <sphere radius="0.0299"/>
+        <sphere radius="0.0499"/>
       </geometry>
     </visual>
@@ -80,9 +80,9 @@
       <origin xyz="0 0 0" rpy="0 1.5707 1.5707"/>
        <geometry>
-        <cylinder length="0.025" radius="0.05"/>
+        <cylinder length="0.05" radius="0.1"/>
       </geometry>
     </visual>
     <inertial>
-      <mass value="3"/>
+      <mass value="5"/>
       <origin xyz="0.0 0 0" rpy=" 0 0 0"/>
       <inertia
@@ -95,5 +95,5 @@
       <origin xyz="0 0 0" rpy="0 1.5707 1.5707"/>
        <geometry>
-        <cylinder length="0.025" radius="0.05"/>
+        <cylinder length="0.05" radius="0.1"/>
       </geometry>
     </collision>
@@ -103,9 +103,9 @@
       <origin xyz="0 0 0" rpy="0 1.5707 1.5707"/>
        <geometry>
-        <cylinder length="0.025" radius="0.05"/>
+        <cylinder length="0.05" radius="0.1"/>
       </geometry>
     </visual>
     <inertial>
-      <mass value="3"/>
+      <mass value="5"/>
       <origin xyz="0.0 0 0" rpy=" 0 0 0"/>
       <inertia
@@ -118,10 +118,10 @@
       <origin xyz="0 0 0" rpy="0 1.5707 1.5707"/>
        <geometry>
-        <cylinder length="0.025" radius="0.05"/>
+        <cylinder length="0.05" radius="0.1"/>
       </geometry>
     </collision>
   </link>
 <joint type="continuous" name="left_wheel_hinge">
-    <origin xyz="0 0.275 0" rpy="0 0 0"/>
+    <origin xyz="0 0.15 0" rpy="0 0 0"/>
     <child link="left_wheel"/>
     <parent link="chassis"/>
@@ -131,5 +131,5 @@
   </joint>
 <joint type="continuous" name="right_wheel_hinge">
-    <origin xyz="0 -0.275 0" rpy="0 0 0"/>
+    <origin xyz="0 -0.15 0" rpy="0 0 0"/>
     <child link="right_wheel"/>
     <parent link="chassis"/>
@@ -162,5 +162,5 @@
 </link>
   <joint name="camera_robot_joint" type="fixed">
-    <origin xyz="0.1 0 0.1" rpy="0 0 0" />
+    <origin xyz="0.2 0 0" rpy="0 0 0" />
     <parent link="chassis"/>
     <child link="camera"/>
@@ -190,5 +190,5 @@
 </link>
   <joint name="hokuyo_joint" type="fixed">
-    <origin xyz=".1 0 .16 " rpy="0 0 0" />
+    <origin xyz=".15 0 .1 " rpy="0 0 0" />
     <parent link="chassis"/>
     <child link="hokuyo"/>

Commit message: final models

File: urdf/udacity_bot.xacro (robot description, xacro)
@@ -9,8 +9,8 @@
   </joint>
   <link name='chassis'>
-    <pose>0 0 0.2 0 0 0</pose>
+    <pose>0 0 0.1 0 0 0</pose>
     <inertial>
-      <mass value="10.0"/>
-      <origin xyz="0.03 0 0" rpy=" 0 0 0"/>
+      <mass value="15"/>
+      <origin xyz="0.0 0 0" rpy=" 0 0 0"/>
       <inertia
           ixx="0.1" ixy="0" ixz="0"
@@ -19,8 +19,8 @@
       />
     </inertial>
-    <collision name='chassis_collision'>
+    <collision name='collision'>
       <origin xyz="0 0 0" rpy=" 0 0 0"/>
       <geometry>
-	<cylinder length="0.03" radius="0.2"/>
+        <box size=".4 .2 .1"/>
       </geometry>
     </collision>
@@ -28,12 +28,18 @@
      <origin xyz="0 0 0" rpy=" 0 0 0"/>
       <geometry>
-	<cylinder length="0.03" radius="0.2"/>
+        <box size=".4 .2 .1"/>
+      </geometry>
+    </visual>
+    <visual name='back_caster_visual'>
+      <origin xyz="-0.15 0 -0.05" rpy=" 0 0 0"/>
+      <geometry>
+        <sphere radius="0.0499"/>
       </geometry>
     </visual>
     <collision name='back_caster_collision'>
-     <origin xyz="-0.2 0 -0.02" rpy=" 0 0 0"/>
-      <geometry>
-        <sphere radius="0.0399"/>
-      </geometry>
+	<origin xyz="-0.15 0 -0.05" rpy=" 0 0 0"/>
+      	<geometry>
+          <sphere radius="0.0499"/>
+      	</geometry>
       <surface>
         <friction>
@@ -47,14 +53,8 @@
       </surface>
     </collision>
-    <visual name='back_caster_visual'>
-     <origin xyz="-0.2 0 -0.02" rpy=" 0 0 0"/>
+    <collision name='front_caster_collision'>
+      <origin xyz="0.15 0 -0.05" rpy=" 0 0 0"/>
       <geometry>
-        <sphere radius="0.0399"/>
-      </geometry>
-    </visual>
-    <collision name='front_caster_collision'>
-     <origin xyz="0.2 0 -0.02" rpy=" 0 0 0"/>
-      <geometry>
-        <sphere radius="0.0399"/>
+        <sphere radius="0.0499"/>
       </geometry>
       <surface>
@@ -70,7 +70,7 @@
     </collision>
     <visual name='front_caster_visual'>
-     <origin xyz="0.2 0 -0.02" rpy=" 0 0 0"/>
+      <origin xyz="0.15 0 -0.05" rpy=" 0 0 0"/>
       <geometry>
-        <sphere radius="0.0399"/>
+        <sphere radius="0.0499"/>
       </geometry>
     </visual>
@@ -80,9 +80,9 @@
       <origin xyz="0 0 0" rpy="0 1.5707 1.5707"/>
        <geometry>
-        <cylinder length="0.025" radius="0.06"/>
+        <cylinder length="0.05" radius="0.1"/>
       </geometry>
     </visual>
     <inertial>
-      <mass value="3"/>
+      <mass value="5"/>
       <origin xyz="0.0 0 0" rpy=" 0 0 0"/>
       <inertia
@@ -95,5 +95,5 @@
       <origin xyz="0 0 0" rpy="0 1.5707 1.5707"/>
        <geometry>
-        <cylinder length="0.025" radius="0.06"/>
+        <cylinder length="0.05" radius="0.1"/>
       </geometry>
     </collision>
@@ -103,9 +103,9 @@
       <origin xyz="0 0 0" rpy="0 1.5707 1.5707"/>
        <geometry>
-        <cylinder length="0.025" radius="0.06"/>
+        <cylinder length="0.05" radius="0.1"/>
       </geometry>
     </visual>
     <inertial>
-      <mass value="3"/>
+      <mass value="5"/>
       <origin xyz="0.0 0 0" rpy=" 0 0 0"/>
       <inertia
@@ -118,10 +118,10 @@
       <origin xyz="0 0 0" rpy="0 1.5707 1.5707"/>
        <geometry>
-        <cylinder length="0.025" radius="0.06"/>
+        <cylinder length="0.05" radius="0.1"/>
       </geometry>
     </collision>
   </link>
 <joint type="continuous" name="left_wheel_hinge">
-    <origin xyz="0 0.226 0" rpy="0 0 0"/>
+    <origin xyz="0 0.15 0" rpy="0 0 0"/>
     <child link="left_wheel"/>
     <parent link="chassis"/>
@@ -131,5 +131,5 @@
   </joint>
 <joint type="continuous" name="right_wheel_hinge">
-    <origin xyz="0 -0.226 0" rpy="0 0 0"/>
+    <origin xyz="0 -0.15 0" rpy="0 0 0"/>
     <child link="right_wheel"/>
     <parent link="chassis"/>
@@ -162,5 +162,5 @@
 </link>
   <joint name="camera_robot_joint" type="fixed">
-    <origin xyz="0.1 0 0.1" rpy="0 0 0" />
+    <origin xyz="0.2 0 0" rpy="0 0 0" />
     <parent link="chassis"/>
     <child link="camera"/>
@@ -190,5 +190,5 @@
 </link>
   <joint name="hokuyo_joint" type="fixed">
-    <origin xyz=".1 0 .16 " rpy="0 0 0" />
+    <origin xyz=".15 0 .1 " rpy="0 0 0" />
     <parent link="chassis"/>
     <child link="hokuyo"/>
